Commit message: Update arm2.urdf.xacro

File: urdf/arm2.urdf.xacro (robot description, xacro)
@@ -77,5 +77,5 @@
         </visual>
         <collision>
-            <origin xyz="0.0 0.0 0.0" rpy="0.0 0.0 0.0"/>
+            <origin xyz="0.0 0.137 -2.15" rpy="0.0 0.0 0.77"/>
             <geometry>
                 <mesh filename="package://arm/meshes/Link_2.stl" scale="0.01 0.01 0.01"/>
@@ -92,5 +92,5 @@
     <link name="link_3">
         <visual>
-            <origin xyz="0.1 -0.79 -2" rpy="-0.0 -0.0 0.77"/>
+            <origin xyz="0.59 -0.61 -2" rpy="-0.1 -0.2 0.77"/>
             <geometry>
                 <mesh filename="package://arm/meshes/Link_3.stl" scale="0.01 0.01 0.01"/>
@@ -114,3 +114,76 @@
         <limit lower="-1.57" upper="1.57" effort="1.0" velocity="1.0"/>
     </joint>
+    <link name="gripper_base">
+        <visual>
+            <origin xyz="1.44 -0.5 -2.505" rpy="-0.2 0.0 3"/>
+            <geometry>
+                <mesh filename="package://arm/meshes/Gripper_Base.stl" scale="0.01 0.01 0.01"/>
+            </geometry>
+            <material name="Grey">
+                <color rgba="0.3 0.3 0.3 1.0"/>
+            </material>
+        </visual>
+        <collision>
+            <origin xyz="0.0 0.0 0.0" rpy="0.0 0.0 0.0"/>
+            <geometry>
+                <mesh filename="package://arm/meshes/Gripper_Base.stl" scale="0.01 0.01 0.01"/>
+            </geometry>
+        </collision>
+    </link>
+    <joint name="gripper_base" type="revolute">
+        <origin xyz="0.19 0.3 0.075" rpy="0.0 0.0 -1.57"/>
+        <parent link="link_3"/>
+        <child link="gripper_base"/>
+        <axis xyz="0.0 1.0 0.0"/>
+        <limit lower="-0.77" upper="2.34" effort="1.0" velocity="1.0"/>
+    </joint>
+    <link name="right_finger">
+        <visual>
+            <origin xyz="-0.2 -0.79 -2.8" rpy="0.0 -0.77 3.14"/>
+            <geometry>
+                <mesh filename="package://arm/meshes/Right_Finger.stl" scale="0.01 0.01 0.01"/>
+            </geometry>
+            <material name="">
+                <color rgba="0.1 0.1 0.4 1.0"/>
+            </material>
+        </visual>
+        <collision>
+            <origin xyz="0.0 0.0 -1.5" rpy="0.0 0.0 3.14"/>
+            <geometry>
+                <mesh filename="package://arm/meshes/Right_Finger.stl" scale="0.01 0.01 0.01"/>
+            </geometry>
+        </collision>
+    </link>
+    <joint name="right" type="revolute">
+        <origin xyz="-0.29 0.09 -0.25" rpy="0.0 -0.77 0.0"/>
+        <parent link="gripper_base"/>
+        <child link="right_finger"/>
+        <axis xyz="0.0 0.0 1.0"/>
+        <limit lower="-1.00" upper="0" effort="0.0" velocity="0.0"/>
+    </joint>
+    <link name="left_finger">
+        <visual>
+            <origin xyz="-0.26 -0.5 -2.8" rpy="0.0 -0.77 3.14"/>
+            <geometry>
+                <mesh filename="package://arm/meshes/Left_Finger.stl" scale="0.01 0.01 0.01"/>
+            </geometry>
+            <material name="Blue">
+                <color rgba="0.1 0.1 0.4 1.0"/>
+            </material>
+        </visual>
+        <collision>
+            <origin xyz="0.0 0.0 0.0" rpy="0.0 0.0 0.0"/>
+            <geometry>
+                <mesh filename="package://arm/meshes/Left_Finger.stl" scale="0.01 0.01 0.01"/>
+            </geometry>
+        </collision>
+    </link>
+    <joint name="left" type="revolute">
+        <origin xyz="-0.29 -0.19 -0.25" rpy="0.0 -0.77 0.0"/>
+        <parent link="gripper_base"/>
+        <child link="left_finger"/>
+        <axis xyz="0.0 0.0 1.0"/>
+        <mimic joint ="right" multiplier ="-1.0"></mimic>
+        <limit lower="0" upper="1" effort="0.0" velocity="0.0"/>
+    </joint>
 </robot>
